Commit message: update_jointconfig

File: src/human_arm_simulation/robot/visual/Human_mockup.xacro (robot description, xacro)
@@ -25,5 +25,5 @@
         <child link="shoulder2"/>
         <axis xyz="0 0 1"/>
-        <limit lower="-0.785" upper="0.785" effort="1000" velocity="0.0"/>
+        <limit lower="0.0" upper="1.57" effort="1000" velocity="0.0"/>
     </joint>
     <!-- Shoulde2 -->
@@ -35,5 +35,5 @@
         <child link="shoulder3"/>
         <axis xyz="0 0 1"/>
-        <limit lower="0" upper="3.14" effort="1000" velocity="0.0"/>
+        <limit lower="0.0" upper="3.14" effort="1000" velocity="0.0"/>
     </joint>
     <!-- Shoulde3 -->
@@ -68,5 +68,5 @@
         <child link="wrist1"/>
         <axis xyz="0 0 1"/>
-        <limit lower="0" upper="2.61" effort="1000" velocity="0.0"/>
+        <limit lower="-1.57" upper="1.57" effort="1000" velocity="0.0"/>
     </joint>
     <!-- Wrist1 -->
@@ -85,5 +85,5 @@
         <child link="wrist2"/>
         <axis xyz="0 0 1"/>
-        <limit lower="0" upper="2.61" effort="1000" velocity="0.0"/>
+        <limit lower="-1.57" upper="1.04" effort="1000" velocity="0.0"/>
     </joint>
     <!-- Wrist2 -->
@@ -95,5 +95,5 @@
         <child link="wrist3"/>
         <axis xyz="0 0 1"/>
-        <limit lower="0" upper="2.61" effort="1000" velocity="0.0"/>
+        <limit lower="-0.34" upper="0.69" effort="1000" velocity="0.0"/>
     </joint>
     <!-- Wrist3 -->

Commit message: edit_xacro

File: src/human_arm_simulation/robot/visual/Human_mockup.xacro (robot description, xacro)
@@ -74,5 +74,5 @@
         <visual>
             <geometry>
-                <cylinder length="0.35" radius="0.05"/>
+                <cylinder length="0.4" radius="0.05"/>
             </geometry>
             <origin xyz="0.0 0.0 -0.2" rpy="0.0 0.0 0.0"/>
