Commit message: Add new urdf and mesh file

File: src/human_arm_simulation/robot/visual/7DOF_robot.xacro (robot description, xacro)
@@ -5,5 +5,5 @@
     <!-- World link Base -->
     <joint name="fixed" type="fixed">
-        <origin xyz="0.0 0.0 1" rpy="0.0 1.57 0.0"/>
+        <origin xyz="0.0 0.0 0.0" rpy="0.0 0.0 0.0"/>
         <parent link="world"/>
         <child link="Base"/>
@@ -15,29 +15,31 @@
                 <mesh filename="package://human_arm_simulation/meshes/Base.STL" />
             </geometry>
+            <origin xyz="-0.16 0.0 0.05" rpy="0.0 0.0 0.0"/>
         </visual>
         <collision>
             <geometry>
-                <mesh filename="package://human_arm_simulation/meshes/Base.STL"/>
+                <mesh filename="package://human_arm_simulation/meshes/Base.STL" />
             </geometry>
+            <origin xyz="-0.16 0.0 0.05" rpy="0.0 0.0 0.0"/>
         </collision>
     </link>
     <!-- q1 -->
     <joint name="q1" type="revolute">
-        <origin xyz="0.0 0.0 0.0" rpy="0.0 0.0 0.0"/>
+        <origin xyz="0.0 0.0 1.0" rpy="1.57 0.0 0.0"/>
         <parent link="Base"/>
-        <child link="Joint1"/>
+        <child link="shoulder1"/>
         <axis xyz="0 0 1"/>
-        <limit lower="-3.14" upper="3.14" effort="1000" velocity="0.0"/>
+        <limit lower="-0.87" upper="3.14" effort="1000" velocity="0.0"/>
     </joint>
-    <!-- Joint1 -->
-    <link name="Joint1">
+    <!-- Shoulde1 -->
+    <link name="shoulder1">
         <visual>
             <geometry>
-                <mesh filename="package://human_arm_simulation/meshes/Joint1.STL" />
+                <mesh filename="package://human_arm_simulation/meshes/Shoulder1.STL"/>
             </geometry>
         </visual>
         <collision>
             <geometry>
-                <mesh filename="package://human_arm_simulation/meshes/Joint1.STL"/>
+                <mesh filename="package://human_arm_simulation/meshes/Shoulder1.STL"/>
             </geometry>
         </collision>
@@ -45,62 +47,53 @@
     <!-- q2 -->
     <joint name="q2" type="revolute">
-        <origin xyz="0.0 0.045 0.045" rpy="-1.57 -1.57 0.0"/>
-        <parent link="Joint1"/>
-        <child link="Joint2"/>
+        <origin xyz="0.0 0.0 0.0" rpy="1.57 -1.57  0.0"/>
+        <parent link="shoulder1"/>
+        <child link="shoulder2"/>
         <axis xyz="0 0 1"/>
-        <limit lower="-3.14" upper="3.14" effort="1000" velocity="0.0"/>
+        <limit lower="0.0" upper="1.57" effort="1000" velocity="0.0"/>
     </joint>
-    <!-- Joint2 -->
-    <link name="Joint2">
+    <!-- Shoulde2 -->
+    <link name="shoulder2"/>
+    <!-- q3 -->
+    <joint name="q3" type="revolute">
+        <origin xyz="0.0 0.0 0.0" rpy="-1.57 -1.57 0.0"/>
+        <parent link="shoulder2"/>
+        <child link="shoulder3"/>
+        <axis xyz="0 0 1"/>
+        <limit lower="0.0" upper="3.14" effort="1000" velocity="0.0"/>
+    </joint>
+    <!-- Shoulde3 -->
+    <link name="shoulder3">
         <visual>
             <geometry>
-                <mesh filename="package://human_arm_simulation/meshes/Joint1.STL" />
+                <mesh filename="package://human_arm_simulation/meshes/Shoulder3.STL"/>
+            </geometry>
+            <origin xyz="0.165 0.0 0.0" rpy="-1.57 0.0 0.0"/>
+        </visual>
+        <collision>
+            <geometry>
+                <mesh filename="package://human_arm_simulation/meshes/Shoulder3.STL"/>
+            </geometry>
+            <origin xyz="0.165 0.0 0.0" rpy="-1.57 0.0 0.0"/>
+        </collision>
+    </link>
+    <!-- q4 -->
+    <joint name="q4" type="revolute">
+        <origin xyz="0.32 0.0 0.0" rpy="-1.57 -1.57 0.0"/>
+        <parent link="shoulder3"/>
+        <child link="elbow"/>
+        <axis xyz="0 0 1"/>
+        <limit lower="0" upper="2.61" effort="1000" velocity="0.0"/>
+    </joint>
+    <!-- Elbow -->
+    <link name="elbow">
+        <visual>
+            <geometry>
+                <mesh filename="package://human_arm_simulation/meshes/Elbow.STL"/>
             </geometry>
         </visual>
         <collision>
             <geometry>
-                <mesh filename="package://human_arm_simulation/meshes/Joint1.STL"/>
-            </geometry>
-        </collision>
-    </link>
-    <!-- q3 -->
-    <joint name="q3" type="revolute">
-        <origin xyz="0.0 0.045 0.045" rpy="-1.57 0.0 0.0"/>
-        <parent link="Joint2"/>
-        <child link="Link1"/>
-        <axis xyz="0 0 1"/>
-        <limit lower="-3.14" upper="3.14" effort="1000" velocity="0.0"/>
-    </joint>
-    <!-- Link1 -->
-    <link name="Link1">
-        <visual>
-            <geometry>
-                <mesh filename="package://human_arm_simulation/meshes/Link1_2.STL" />
-            </geometry>
-        </visual>
-        <collision>
-            <geometry>
-                <mesh filename="package://human_arm_simulation/meshes/Link1_2.STL"/>
-            </geometry>
-        </collision>
-    </link>
-    <!-- q4 -->
-    <joint name="q4" type="revolute">
-        <origin xyz="0.0 0.045 0.345" rpy="-1.57 -1.57 0.0"/>
-        <parent link="Link1"/>
-        <child link="Link2"/>
-        <axis xyz="0 0 1"/>
-        <limit lower="-3.14" upper="3.14" effort="1000" velocity="0.0"/>
-    </joint>
-    <!-- Link2 -->
-    <link name="Link2">
-        <visual>
-            <geometry>
-                <mesh filename="package://human_arm_simulation/meshes/Link1_1.STL" />
-            </geometry>
-        </visual>
-        <collision>
-            <geometry>
-                <mesh filename="package://human_arm_simulation/meshes/Link1_1.STL"/>
+                <mesh filename="package://human_arm_simulation/meshes/Elbow.STL"/>
             </geometry>
         </collision>
@@ -108,63 +101,56 @@
     <!-- q5 -->
     <joint name="q5" type="revolute">
-        <origin xyz="0.345 0.0 0.045" rpy="0.0 1.57 0.0"/>
-        <parent link="Link2"/>
-        <child link="Joint3"/>
+        <origin xyz="0.0 0.355 0.0" rpy="-1.57 0.0 0.0"/>
+        <parent link="elbow"/>
+        <child link="wrist1"/>
         <axis xyz="0 0 1"/>
-        <limit lower="-3.14" upper="3.14" effort="1000" velocity="0.0"/>
+        <limit lower="-1.57" upper="1.57" effort="1000" velocity="0.0"/>
     </joint>
-    <!-- Joint3 -->
-    <link name="Joint3">
+    <!-- Wrist1 -->
+    <link name="wrist1">
         <visual>
             <geometry>
-                <mesh filename="package://human_arm_simulation/meshes/Joint1.STL" />
+                <mesh filename="package://human_arm_simulation/meshes/Wrist1.STL"/>
             </geometry>
+            <origin xyz="0.0 0.0 -0.2" rpy="0.0 0.0 -1.57"/>
         </visual>
         <collision>
             <geometry>
-                <mesh filename="package://human_arm_simulation/meshes/Joint1.STL"/>
+                <mesh filename="package://human_arm_simulation/meshes/Wrist1.STL"/>
             </geometry>
+            <origin xyz="0.0 0.0 -0.2" rpy="0.0 0.0 -1.57"/>
         </collision>
     </link>
     <!-- q6 -->
     <joint name="q6" type="revolute">
-        <origin xyz="0.0 0.045 0.045" rpy="-1.57 0.0 0.0"/>
-        <parent link="Joint3"/>
-        <child link="Joint4"/>
+        <origin xyz="0.0 0.0 -0.05" rpy="1.57 -1.57 0.0"/>
+        <parent link="wrist1"/>
+        <child link="wrist2"/>
         <axis xyz="0 0 1"/>
-        <limit lower="-3.14" upper="3.14" effort="1000" velocity="0.0"/>
+        <limit lower="-1.57" upper="1.04" effort="1000" velocity="0.0"/>
     </joint>
-    <!-- Joint4 -->
-    <link name="Joint4">
+    <!-- Wrist2 -->
+    <link name="wrist2"/>
+     <!-- q7 -->
+    <joint name="q7" type="revolute">
+        <origin xyz="0.0 0.0 0.0" rpy="1.57 0.0 0.0"/>
+        <parent link="wrist2"/>
+        <child link="wrist3"/>
+        <axis xyz="0 0 1"/>
+        <limit lower="-0.34" upper="0.69" effort="1000" velocity="0.0"/>
+    </joint>
+    <!-- Wrist3 -->
+    <link name="wrist3">
         <visual>
             <geometry>
-                <mesh filename="package://human_arm_simulation/meshes/Joint1.STL" />
+                <mesh filename="package://human_arm_simulation/meshes/Wrist3.STL"/>
             </geometry>
+            <origin xyz="0.0 0.0 0.0" rpy="-1.57 0.0 0.0"/>
         </visual>
         <collision>
             <geometry>
-                <mesh filename="package://human_arm_simulation/meshes/Joint1.STL"/>
+                <mesh filename="package://human_arm_simulation/meshes/Wrist3.STL"/>
             </geometry>
-        </collision>
-    </link>
-    <!-- q7 -->
-    <joint name="q7" type="revolute">
-        <origin xyz="0.0 0.045 0.045" rpy="-1.57 0.0 0.0"/>
-        <parent link="Joint4"/>
-        <child link="Gripper"/>
-        <axis xyz="0 0 1"/>
-        <limit lower="-3.14" upper="3.14" effort="1000" velocity="0.0"/>
-    </joint>
-    <!-- Gripper -->
-    <link name="Gripper">
-        <visual>
-            <geometry>
-                <mesh filename="package://human_arm_simulation/meshes/Gripper.STL" />
-            </geometry>
-        </visual>
-        <collision>
-            <geometry>
-                <mesh filename="package://human_arm_simulation/meshes/Gripper.STL"/>
-            </geometry>
+            <origin xyz="0.0 0.0 0.0" rpy="-1.57 0.0 0.0"/>
         </collision>
     </link>

Commit message: Fix urdf file

File: src/human_arm_simulation/robot/visual/7DOF_robot.xacro (robot description, xacro)
@@ -13,13 +13,13 @@
         <visual>
             <geometry>
-                <mesh filename="package://human_arm_simulation/meshes/Base.STL" />
+                <mesh filename="../meshes/Base.STL" />
             </geometry>
-            <origin xyz="-0.16 0.0 0.05" rpy="0.0 0.0 0.0"/>
+            <origin xyz="0.0 0.16 0.0" rpy="0.0 0.0 -1.57"/>
         </visual>
         <collision>
             <geometry>
-                <mesh filename="package://human_arm_simulation/meshes/Base.STL" />
+                <mesh filename="../meshes/Base.STL" />
             </geometry>
-            <origin xyz="-0.16 0.0 0.05" rpy="0.0 0.0 0.0"/>
+            <origin xyz="0.0 0.16 0.0" rpy="0.0 0.0 -1.57"/>
         </collision>
     </link>
@@ -36,10 +36,10 @@
         <visual>
             <geometry>
-                <mesh filename="package://human_arm_simulation/meshes/Shoulder1.STL"/>
+                <mesh filename="../meshes/Shoulder1.STL"/>
             </geometry>
         </visual>
         <collision>
             <geometry>
-                <mesh filename="package://human_arm_simulation/meshes/Shoulder1.STL"/>
+                <mesh filename="../meshes/Shoulder1.STL"/>
             </geometry>
         </collision>
@@ -67,5 +67,5 @@
         <visual>
             <geometry>
-                <mesh filename="package://human_arm_simulation/meshes/Shoulder3.STL"/>
+                <mesh filename="../meshes/Shoulder3.STL"/>
             </geometry>
             <origin xyz="0.165 0.0 0.0" rpy="-1.57 0.0 0.0"/>
@@ -73,5 +73,5 @@
         <collision>
             <geometry>
-                <mesh filename="package://human_arm_simulation/meshes/Shoulder3.STL"/>
+                <mesh filename="../meshes/Shoulder3.STL"/>
             </geometry>
             <origin xyz="0.165 0.0 0.0" rpy="-1.57 0.0 0.0"/>
@@ -90,10 +90,10 @@
         <visual>
             <geometry>
-                <mesh filename="package://human_arm_simulation/meshes/Elbow.STL"/>
+                <mesh filename="../meshes/Elbow.STL"/>
             </geometry>
         </visual>
         <collision>
             <geometry>
-                <mesh filename="package://human_arm_simulation/meshes/Elbow.STL"/>
+                <mesh filename="../meshes/Elbow.STL"/>
             </geometry>
         </collision>
@@ -111,5 +111,5 @@
         <visual>
             <geometry>
-                <mesh filename="package://human_arm_simulation/meshes/Wrist1.STL"/>
+                <mesh filename="../meshes/Wrist1.STL"/>
             </geometry>
             <origin xyz="0.0 0.0 -0.2" rpy="0.0 0.0 -1.57"/>
@@ -117,5 +117,5 @@
         <collision>
             <geometry>
-                <mesh filename="package://human_arm_simulation/meshes/Wrist1.STL"/>
+                <mesh filename="../meshes/Wrist1.STL"/>
             </geometry>
             <origin xyz="0.0 0.0 -0.2" rpy="0.0 0.0 -1.57"/>
@@ -144,13 +144,13 @@
         <visual>
             <geometry>
-                <mesh filename="package://human_arm_simulation/meshes/Wrist3.STL"/>
+                <mesh filename="../meshes/Wrist3.STL"/>
             </geometry>
-            <origin xyz="0.0 0.0 0.0" rpy="-1.57 0.0 0.0"/>
+            <origin xyz="0.0 0.0 0.0" rpy="0 0.0 0.0"/>
         </visual>
         <collision>
             <geometry>
-                <mesh filename="package://human_arm_simulation/meshes/Wrist3.STL"/>
+                <mesh filename="../meshes/Wrist3.STL"/>
             </geometry>
-            <origin xyz="0.0 0.0 0.0" rpy="-1.57 0.0 0.0"/>
+            <origin xyz="0.0 0.0 0.0" rpy="0 0.0 0.0"/>
         </collision>
     </link>

Commit message: Fix urdf path

File: src/human_arm_simulation/robot/visual/7DOF_robot.xacro (robot description, xacro)
@@ -13,5 +13,5 @@
         <visual>
             <geometry>
-                <mesh filename="../meshes/Base.STL" />
+                <mesh filename="package://human_arm_simulation/meshes/Base.STL" />
             </geometry>
             <origin xyz="0.0 0.16 0.0" rpy="0.0 0.0 -1.57"/>
@@ -19,5 +19,5 @@
         <collision>
             <geometry>
-                <mesh filename="../meshes/Base.STL" />
+                <mesh filename="package://human_arm_simulation/meshes/Base.STL" />
             </geometry>
             <origin xyz="0.0 0.16 0.0" rpy="0.0 0.0 -1.57"/>
@@ -36,10 +36,10 @@
         <visual>
             <geometry>
-                <mesh filename="../meshes/Shoulder1.STL"/>
+                <mesh filename="package://human_arm_simulation/meshes/Shoulder1.STL"/>
             </geometry>
         </visual>
         <collision>
             <geometry>
-                <mesh filename="../meshes/Shoulder1.STL"/>
+                <mesh filename="package://human_arm_simulation/meshes/Shoulder1.STL"/>
             </geometry>
         </collision>
@@ -67,5 +67,5 @@
         <visual>
             <geometry>
-                <mesh filename="../meshes/Shoulder3.STL"/>
+                <mesh filename="package://human_arm_simulation/meshes/Shoulder3.STL"/>
             </geometry>
             <origin xyz="0.165 0.0 0.0" rpy="-1.57 0.0 0.0"/>
@@ -73,5 +73,5 @@
         <collision>
             <geometry>
-                <mesh filename="../meshes/Shoulder3.STL"/>
+                <mesh filename="package://human_arm_simulation/meshes/Shoulder3.STL"/>
             </geometry>
             <origin xyz="0.165 0.0 0.0" rpy="-1.57 0.0 0.0"/>
@@ -90,10 +90,10 @@
         <visual>
             <geometry>
-                <mesh filename="../meshes/Elbow.STL"/>
+                <mesh filename="package://human_arm_simulation/meshes/Elbow.STL"/>
             </geometry>
         </visual>
         <collision>
             <geometry>
-                <mesh filename="../meshes/Elbow.STL"/>
+                <mesh filename="package://human_arm_simulation/meshes/Elbow.STL"/>
             </geometry>
         </collision>
@@ -111,5 +111,5 @@
         <visual>
             <geometry>
-                <mesh filename="../meshes/Wrist1.STL"/>
+                <mesh filename="package://human_arm_simulation/meshes/Wrist1.STL"/>
             </geometry>
             <origin xyz="0.0 0.0 -0.2" rpy="0.0 0.0 -1.57"/>
@@ -117,5 +117,5 @@
         <collision>
             <geometry>
-                <mesh filename="../meshes/Wrist1.STL"/>
+                <mesh filename="package://human_arm_simulation/meshes/Wrist1.STL"/>
             </geometry>
             <origin xyz="0.0 0.0 -0.2" rpy="0.0 0.0 -1.57"/>
@@ -144,5 +144,5 @@
         <visual>
             <geometry>
-                <mesh filename="../meshes/Wrist3.STL"/>
+                <mesh filename="package://human_arm_simulation/meshes/Wrist3.STL"/>
             </geometry>
             <origin xyz="0.0 0.0 0.0" rpy="0 0.0 0.0"/>
@@ -150,5 +150,5 @@
         <collision>
             <geometry>
-                <mesh filename="../meshes/Wrist3.STL"/>
+                <mesh filename="package://human_arm_simulation/meshes/Wrist3.STL"/>
             </geometry>
             <origin xyz="0.0 0.0 0.0" rpy="0 0.0 0.0"/>
