Commit message: Update New Can 'Correct Axis'

File: urdf/7DOF_robot copy.URDF (robot description, URDF)
Before this commit: robot 7DOF_ROBOT, 9 links, 8 joints
Links:
- removed link wrist2
- removed link wrist3
- link elbow: geometry visual mesh filename=../meshes/Elbow.STL
- link shoulder1: geometry visual mesh filename=../meshes/Shoulder1.STL
- link shoulder3: geometry visual mesh filename=../meshes/Shoulder3.STL
- link wrist1: geometry visual mesh filename=../meshes/Wrist1.STL
Joints:
- removed joint q6
- removed joint q7
- joint q1: origin xyz=0.0 0.0 1.0 rpy=1.57 0.0 0.0 -> xyz=0.15 0.0 0.95 rpy=1.57 0.0 0.0
- joint q4: origin xyz=0.32 0.0 0.0 rpy=-1.57 -1.57 0.0 -> xyz=0.3 0.0 0.0 rpy=-1.57 -1.57 0.0
- joint q5: origin xyz=0.0 0.355 0.0 rpy=-1.57 0.0 0.0 -> xyz=0.0 0.35 0.0 rpy=-1.57 0.0 0.0

File: urdf/Human_mockup.xacro (robot description, xacro)
@@ -3,29 +3,8 @@
     <!-- World -->
     <link name="world"/>
-    <!-- World link Base -->
-    <joint name="fixed" type="fixed">
-        <origin xyz="0.0 0.0 0.0" rpy="0.0 0.0 0.0"/>
-        <parent link="world"/>
-        <child link="Base"/>
-    </joint>
-    <!-- Base  -->
-    <link name="Base">
-        <visual>
-            <geometry>
-                <mesh filename="../meshes/Base.STL" />
-            </geometry>
-            <origin xyz="-0.16 0.0 0.05" rpy="0.0 0.0 0.0"/>
-        </visual>
-        <collision>
-            <geometry>
-                <mesh filename="../meshes/Base.STL" />
-            </geometry>
-            <origin xyz="-0.16 0.0 0.05" rpy="0.0 0.0 0.0"/>
-        </collision>
-    </link>
     <!-- q1 -->
     <joint name="q1" type="revolute">
         <origin xyz="0.0 0.0 1.0" rpy="1.57 0.0 0.0"/>
-        <parent link="Base"/>
+        <parent link="world"/>
         <child link="shoulder1"/>
         <axis xyz="0 0 1"/>
@@ -36,12 +15,7 @@
         <visual>
             <geometry>
-                <mesh filename="../meshes/Shoulder1.STL"/>
+                <sphere radius="0.05"/>
             </geometry>
         </visual>
-        <collision>
-            <geometry>
-                <mesh filename="../meshes/Shoulder1.STL"/>
-            </geometry>
-        </collision>
     </link>
     <!-- q2 -->
@@ -67,18 +41,12 @@
         <visual>
             <geometry>
-                <mesh filename="../meshes/Shoulder3.STL"/>
+                <cylinder length="0.4" radius="0.05"/>
             </geometry>
-            <origin xyz="0.165 0.0 0.0" rpy="-1.57 0.0 0.0"/>
+            <origin xyz="0.2 0.0 0.0" rpy="0.0 1.57 0.0"/>
         </visual>
-        <collision>
-            <geometry>
-                <mesh filename="../meshes/Shoulder3.STL"/>
-            </geometry>
-            <origin xyz="0.165 0.0 0.0" rpy="-1.57 0.0 0.0"/>
-        </collision>
     </link>
     <!-- q4 -->
     <joint name="q4" type="revolute">
-        <origin xyz="0.32 0.0 0.0" rpy="-1.57 -1.57 0.0"/>
+        <origin xyz="0.4 0.0 0.0" rpy="-1.57 -1.57 0.0"/>
         <parent link="shoulder3"/>
         <child link="elbow"/>
@@ -90,16 +58,11 @@
         <visual>
             <geometry>
-                <mesh filename="../meshes/Elbow.STL"/>
+                <sphere radius="0.05"/>
             </geometry>
         </visual>
-        <collision>
-            <geometry>
-                <mesh filename="../meshes/Elbow.STL"/>
-            </geometry>
-        </collision>
     </link>
     <!-- q5 -->
     <joint name="q5" type="revolute">
-        <origin xyz="0.0 0.355 0.0" rpy="-1.57 0.0 0.0"/>
+        <origin xyz="0.0 0.4 0.0" rpy="-1.57 0.0 0.0"/>
         <parent link="elbow"/>
         <child link="wrist1"/>
@@ -111,14 +74,8 @@
         <visual>
             <geometry>
-                <mesh filename="../meshes/Wrist1.STL"/>
+                <cylinder length="0.35" radius="0.05"/>
             </geometry>
-            <origin xyz="0.0 0.0 -0.2" rpy="0.0 0.0 -1.57"/>
+            <origin xyz="0.0 0.0 -0.2" rpy="0.0 0.0 0.0"/>
         </visual>
-        <collision>
-            <geometry>
-                <mesh filename="../meshes/Wrist1.STL"/>
-            </geometry>
-            <origin xyz="0.0 0.0 -0.2" rpy="0.0 0.0 -1.57"/>
-        </collision>
     </link>
     <!-- q6 -->
@@ -134,5 +91,5 @@
      <!-- q7 -->
     <joint name="q7" type="revolute">
-        <origin xyz="-0.05 0.0 0.0" rpy="1.57 0.0 0.0"/>
+        <origin xyz="0.0 0.0 0.0" rpy="1.57 0.0 0.0"/>
         <parent link="wrist2"/>
         <child link="wrist3"/>
@@ -142,16 +99,9 @@
     <!-- Wrist3 -->
     <link name="wrist3">
-        <visual>
+            <visual>
             <geometry>
-                <mesh filename="../meshes/Wrist3.STL"/>
+                <box size="0.2 0.1 0.1"/>
             </geometry>
-            <origin xyz="0 0.0 0.0" rpy="-1.57 0.0 0.0"/>
         </visual>
-        <collision>
-            <geometry>
-                <mesh filename="../meshes/Wrist3.STL"/>
-            </geometry>
-            <origin xyz="0 0.0 0.0" rpy="-1.57 0.0 0.0"/>
-        </collision>
     </link>
 </robot>
