Commit message: 7Dof URDF 7DoF but wrong axis...

File: urdf/7DOF_robot.URDF (robot description, URDF)
Before this commit: robot 7DOF_ROBOT, 0 links, 0 joints
Links:
- added link Base; collision mesh filename=../meshes/Base.STL; visual mesh filename=../meshes/Base.STL
- added link Gripper; collision mesh filename=../meshes/Gripper.STL; visual mesh filename=../meshes/Gripper.STL
- added link Joint1; collision mesh filename=../meshes/Joint1.STL; visual mesh filename=../meshes/Joint1.STL
- added link Joint2; collision mesh filename=../meshes/Joint1.STL; visual mesh filename=../meshes/Joint1.STL
- added link Joint3; collision mesh filename=../meshes/Joint1.STL; visual mesh filename=../meshes/Joint1.STL
- added link Joint4; collision mesh filename=../meshes/Joint1.STL; visual mesh filename=../meshes/Joint1.STL
- added link Link1; collision mesh filename=../meshes/Link1.STL; visual mesh filename=../meshes/Link1.STL
- added link Link2; collision mesh filename=../meshes/Link1.STL; visual mesh filename=../meshes/Link1.STL
- added link world
Joints:
- added joint fixed: type fixed, parent world, child Base, origin xyz=0.0 0.0 1 rpy=0.0 1.57 0.0
- added joint q1: type revolute, parent Base, child Joint1, origin xyz=0.0 0.0 0.0 rpy=0.0 0.0 0.0, axis 0 0 1, limit lower=-3.14 upper=3.14 effort=1000 velocity=0.0
- added joint q2: type revolute, parent Joint1, child Link1, origin xyz=0.0 0.045 0.045 rpy=-1.57 0.0 0.0, axis 0 0 1, limit lower=-3.14 upper=3.14 effort=1000 velocity=0.0
- added joint q3: type revolute, parent Link1, child Joint2, origin xyz=0.345 0.0 0.045 rpy=0.0 -1.57 3.14, axis 0 0 1, limit lower=-3.14 upper=3.14 effort=1000 velocity=0.0
- added joint q4: type revolute, parent Joint2, child Link2, origin xyz=0.0 0.045 0.045 rpy=-1.57 -1.57 0.0, axis 0 0 1, limit lower=-3.14 upper=3.14 effort=1000 velocity=0.0
- added joint q5: type revolute, parent Link2, child Joint3, origin xyz=0.345 0.0 0.045 rpy=0.0 1.57 0.0, axis 0 0 1, limit lower=-3.14 upper=3.14 effort=1000 velocity=0.0
- added joint q6: type revolute, parent Joint3, child Joint4, origin xyz=0.0 0.045 0.045 rpy=-1.57 1.57 0.0, axis 0 0 1, limit lower=-3.14 upper=3.14 effort=1000 velocity=0.0
- added joint q7: type revolute, parent Joint4, child Gripper, origin xyz=0.0 0.045 0.045 rpy=-1.57 1.57 0.0, axis 0 0 1, limit lower=-3.14 upper=3.14 effort=1000 velocity=0.0

Commit message: New URDF

File: urdf/7DOF_robot.URDF (robot description, URDF)
Before this commit: robot 7DOF_ROBOT, 9 links, 8 joints
Links:
- link Link1: geometry collision mesh filename=../meshes/Link1_2.STL; visual mesh filename=../meshes/Link1_2.STL
- link Link2: geometry collision mesh filename=../meshes/Link1_1.STL; visual mesh filename=../meshes/Link1_1.STL
Joints:
- joint q2: child Link1 -> Joint2; origin xyz=0.0 0.045 0.045 rpy=-1.57 0.0 0.0 -> xyz=0.0 0.045 0.045 rpy=-1.57 -1.57 0.0
- joint q3: child Joint2 -> Link1; origin xyz=0.345 0.0 0.045 rpy=0.0 -1.57 3.14 -> xyz=0.0 0.045 0.045 rpy=-1.57 0.0 0.0; parent Link1 -> Joint2
- joint q4: origin xyz=0.0 0.045 0.045 rpy=-1.57 -1.57 0.0 -> xyz=0.0 0.045 0.345 rpy=-1.57 -1.57 0.0; parent Joint2 -> Link1
- joint q6: origin xyz=0.0 0.045 0.045 rpy=-1.57 1.57 0.0 -> xyz=0.0 0.045 0.045 rpy=-1.57 0.0 0.0
- joint q7: origin xyz=0.0 0.045 0.045 rpy=-1.57 1.57 0.0 -> xyz=0.0 0.045 0.045 rpy=-1.57 0.0 0.0

Commit message: fix q6 axis

File: urdf/7DOF_robot.URDF (robot description, URDF)
Before this commit: robot 7DOF_ROBOT, 9 links, 8 joints
Joints:
- joint q6: origin xyz=0.0 0.0 0.0 rpy=1.57 -1.57 0.0 -> xyz=0.0 0.0 -0.05 rpy=1.57 -1.57 0.0

Commit message: fix q6 round 2

File: urdf/7DOF_robot.URDF (robot description, URDF)
Before this commit: robot 7DOF_ROBOT, 9 links, 8 joints
Joints:
- joint q7: origin xyz=-0.05 0.0 0.0 rpy=1.57 0.0 0.0 -> xyz=0.0 0.0 0.0 rpy=1.57 0.0 0.0
